Commit message: Add files via upload

File: voxbot/urdf/voxbot.urdf (robot description, URDF)
Before this commit: robot voxbot, 46 links, 45 joints
Links:
- added link imu_link
- added link sensor_link
Joints:
- added joint imu_joint: type fixed, parent base_link, child imu_link, origin xyz=0.0 0 0.068 rpy=0 0 0
- added joint sensor_joint: type fixed, parent dummy_link, child sensor_link, origin xyz=0.0 0.0 0.05 rpy=0 0 0
