Commit message: neccessary changes

File: vox_description/urdf/voxbot.urdf (robot description, URDF)
Before this commit: robot voxbot, 46 links, 45 joints
Links:
- link b_wheel_link: geometry collision mesh filename=package://vox_description/meshes/base_link.STL; visual mesh filename=package://vox_description/meshes/base_link.STL
- link base_link: geometry collision mesh filename=package://vox_description/meshes/chassis_link.STL; visual mesh filename=package://vox_description/meshes/chassis_link.STL
- link f_wheel_link: geometry collision mesh filename=package://vox_description/meshes/base_link.STL; visual mesh filename=package://vox_description/meshes/base_link.STL
- link l_wheel_link: geometry collision mesh filename=package://vox_description/meshes/base_link.STL; visual mesh filename=package://vox_description/meshes/base_link.STL
- link r_wheel_link: geometry collision mesh filename=package://vox_description/meshes/base_link.STL; visual mesh filename=package://vox_description/meshes/base_link.STL
- link rb10_link: geometry collision mesh filename=package://vox_description/meshes/r10_link.STL; visual mesh filename=package://vox_description/meshes/r10_link.STL
- link rb1_link: geometry collision mesh filename=package://vox_description/meshes/r1_link.STL; visual mesh filename=package://vox_description/meshes/r1_link.STL
- link rb2_link: geometry collision mesh filename=package://vox_description/meshes/r2_link.STL; visual mesh filename=package://vox_description/meshes/r2_link.STL
- link rb3_link: geometry collision mesh filename=package://vox_description/meshes/r3_link.STL; visual mesh filename=package://vox_description/meshes/r3_link.STL
- link rb4_link: geometry collision mesh filename=package://vox_description/meshes/r4_link.STL; visual mesh filename=package://vox_description/meshes/r4_link.STL
- link rb5_link: geometry collision mesh filename=package://vox_description/meshes/r5_link.STL; visual mesh filename=package://vox_description/meshes/r5_link.STL
- link rb6_link: geometry collision mesh filename=package://vox_description/meshes/r6_link.STL; visual mesh filename=package://vox_description/meshes/r6_link.STL
- link rb7_link: geometry collision mesh filename=package://vox_description/meshes/r7_link.STL; visual mesh filename=package://vox_description/meshes/r7_link.STL
- link rb8_link: geometry collision mesh filename=package://vox_description/meshes/r8_link.STL; visual mesh filename=package://vox_description/meshes/r8_link.STL
- link rb9_link: geometry collision mesh filename=package://vox_description/meshes/r9_link.STL; visual mesh filename=package://vox_description/meshes/r9_link.STL
- link rf10_link: geometry collision mesh filename=package://vox_description/meshes/r10_link.STL; visual mesh filename=package://vox_description/meshes/r10_link.STL
- link rf1_link: geometry collision mesh filename=package://vox_description/meshes/r1_link.STL; visual mesh filename=package://vox_description/meshes/r1_link.STL
- link rf2_link: geometry collision mesh filename=package://vox_description/meshes/r2_link.STL; visual mesh filename=package://vox_description/meshes/r2_link.STL
- link rf3_link: geometry collision mesh filename=package://vox_description/meshes/r3_link.STL; visual mesh filename=package://vox_description/meshes/r3_link.STL
- link rf4_link: geometry collision mesh filename=package://vox_description/meshes/r4_link.STL; visual mesh filename=package://vox_description/meshes/r4_link.STL
- link rf5_link: geometry collision mesh filename=package://vox_description/meshes/r5_link.STL; visual mesh filename=package://vox_description/meshes/r5_link.STL
- link rf6_link: geometry collision mesh filename=package://vox_description/meshes/r6_link.STL; visual mesh filename=package://vox_description/meshes/r6_link.STL
- link rf7_link: geometry collision mesh filename=package://vox_description/meshes/r7_link.STL; visual mesh filename=package://vox_description/meshes/r7_link.STL
- link rf8_link: geometry collision mesh filename=package://vox_description/meshes/r8_link.STL; visual mesh filename=package://vox_description/meshes/r8_link.STL
- link rf9_link: geometry collision mesh filename=package://vox_description/meshes/r9_link.STL; visual mesh filename=package://vox_description/meshes/r9_link.STL
- link rl10_link: geometry collision mesh filename=package://vox_description/meshes/r10_link.STL; visual mesh filename=package://vox_description/meshes/r10_link.STL
- link rl1_link: geometry collision mesh filename=package://vox_description/meshes/r1_link.STL; visual mesh filename=package://vox_description/meshes/r1_link.STL
- link rl2_link: geometry collision mesh filename=package://vox_description/meshes/r2_link.STL; visual mesh filename=package://vox_description/meshes/r2_link.STL
- link rl3_link: geometry collision mesh filename=package://vox_description/meshes/r3_link.STL; visual mesh filename=package://vox_description/meshes/r3_link.STL
- link rl4_link: geometry collision mesh filename=package://vox_description/meshes/r4_link.STL; visual mesh filename=package://vox_description/meshes/r4_link.STL
- link rl5_link: geometry collision mesh filename=package://vox_description/meshes/r5_link.STL; visual mesh filename=package://vox_description/meshes/r5_link.STL
- link rl6_link: geometry collision mesh filename=package://vox_description/meshes/r6_link.STL; visual mesh filename=package://vox_description/meshes/r6_link.STL
- link rl7_link: geometry collision mesh filename=package://vox_description/meshes/r7_link.STL; visual mesh filename=package://vox_description/meshes/r7_link.STL
- link rl8_link: geometry collision mesh filename=package://vox_description/meshes/r8_link.STL; visual mesh filename=package://vox_description/meshes/r8_link.STL
- link rl9_link: geometry collision mesh filename=package://vox_description/meshes/r9_link.STL; visual mesh filename=package://vox_description/meshes/r9_link.STL
- link rr10_link: geometry collision mesh filename=package://vox_description/meshes/r10_link.STL; visual mesh filename=package://vox_description/meshes/r10_link.STL
- link rr1_link: geometry collision mesh filename=package://vox_description/meshes/r1_link.STL; visual mesh filename=package://vox_description/meshes/r1_link.STL
- link rr2_link: geometry collision mesh filename=package://vox_description/meshes/r2_link.STL; visual mesh filename=package://vox_description/meshes/r2_link.STL
- link rr3_link: geometry collision mesh filename=package://vox_description/meshes/r3_link.STL; visual mesh filename=package://vox_description/meshes/r3_link.STL
- link rr4_link: geometry collision mesh filename=package://vox_description/meshes/r4_link.STL; visual mesh filename=package://vox_description/meshes/r4_link.STL
- link rr5_link: geometry collision mesh filename=package://vox_description/meshes/r5_link.STL; visual mesh filename=package://vox_description/meshes/r5_link.STL
- link rr6_link: geometry collision mesh filename=package://vox_description/meshes/r6_link.STL; visual mesh filename=package://vox_description/meshes/r6_link.STL
- link rr7_link: geometry collision mesh filename=package://vox_description/meshes/r7_link.STL; visual mesh filename=package://vox_description/meshes/r7_link.STL
- link rr8_link: geometry collision mesh filename=package://vox_description/meshes/r8_link.STL; visual mesh filename=package://vox_description/meshes/r8_link.STL
- link rr9_link: geometry collision mesh filename=package://vox_description/meshes/r9_link.STL; visual mesh filename=package://vox_description/meshes/r9_link.STL

Commit message: fixed odom

File: vox_description/urdf/voxbot.urdf (robot description, URDF)
Before this commit: robot voxbot, 46 links, 45 joints
Links:
- added link imu_link
- added link sensor_link
Joints:
- added joint imu_joint: type fixed, parent dummy_link, child imu_link, origin xyz=0.0 0 0.068 rpy=0 0 0
- added joint sensor_joint: type fixed, parent dummy_link, child sensor_link, origin xyz=0.0 0.0 0.05 rpy=0 0 0
- joint b_wheel2base_joint: origin xyz=0 -0.015 -0.1758 rpy=-3.1457 0 0.0162722351660208 -> xyz=-0.1758 -0.015 0 rpy=-3.1416 -1.5561 -3.14
- joint f_wheel2base_joint: origin xyz=0 -0.015 0.1758 rpy=0 0 3.1285 -> xyz=0.1758 -0.015 0 rpy=-3.1416 -1.5344 0
- joint l_wheel2base_joint: origin xyz=-0.1758 -0.015 0 rpy=-3.1416 -1.5561 -3.14 -> xyz=0 -0.015 0.1758 rpy=0 0 3.1285
- joint r_wheel2base_joint: origin xyz=0.1758 -0.015 0 rpy=-3.1416 -1.5344 0 -> xyz=0 -0.015 -0.1758 rpy=-3.1457 0 0.0162722351660208

Commit message: Improved RTF using reduced meshes

File: vox_description/urdf/voxbot.urdf (robot description, URDF)
Before this commit: robot voxbot, 48 links, 47 joints
Links:
- link b_wheel_link: geometry collision mesh filename=package://vox_description/meshes/base_link.stl; visual mesh filename=package://vox_description/meshes/base_link.stl
- link base_link: geometry collision mesh filename=package://vox_description/meshes/chassis_link.stl; visual mesh filename=package://vox_description/meshes/chassis_link.stl
- link f_wheel_link: geometry collision mesh filename=package://vox_description/meshes/base_link.stl; visual mesh filename=package://vox_description/meshes/base_link.stl
- link l_wheel_link: geometry collision mesh filename=package://vox_description/meshes/base_link.stl; visual mesh filename=package://vox_description/meshes/base_link.stl
- link r_wheel_link: geometry collision mesh filename=package://vox_description/meshes/base_link.stl; visual mesh filename=package://vox_description/meshes/base_link.stl
- link rb10_link: geometry collision mesh filename=package://vox_description/meshes/r10_link.stl; visual mesh filename=package://vox_description/meshes/r10_link.stl
- link rb1_link: geometry collision mesh filename=package://vox_description/meshes/r1_link.stl; visual mesh filename=package://vox_description/meshes/r1_link.stl
- link rb2_link: geometry collision mesh filename=package://vox_description/meshes/r2_link.stl; visual mesh filename=package://vox_description/meshes/r2_link.stl
- link rb3_link: geometry collision mesh filename=package://vox_description/meshes/r3_link.stl; visual mesh filename=package://vox_description/meshes/r3_link.stl
- link rb4_link: geometry collision mesh filename=package://vox_description/meshes/r4_link.stl; visual mesh filename=package://vox_description/meshes/r4_link.stl
- link rb5_link: geometry collision mesh filename=package://vox_description/meshes/r5_link.stl; visual mesh filename=package://vox_description/meshes/r5_link.stl
- link rb6_link: geometry collision mesh filename=package://vox_description/meshes/r6_link.stl; visual mesh filename=package://vox_description/meshes/r6_link.stl
- link rb7_link: geometry collision mesh filename=package://vox_description/meshes/r7_link.stl; visual mesh filename=package://vox_description/meshes/r7_link.stl
- link rb8_link: geometry collision mesh filename=package://vox_description/meshes/r8_link.stl; visual mesh filename=package://vox_description/meshes/r8_link.stl
- link rb9_link: geometry collision mesh filename=package://vox_description/meshes/r9_link.stl; visual mesh filename=package://vox_description/meshes/r9_link.stl
- link rf10_link: geometry collision mesh filename=package://vox_description/meshes/r10_link.stl; visual mesh filename=package://vox_description/meshes/r10_link.stl
- link rf1_link: geometry collision mesh filename=package://vox_description/meshes/r1_link.stl; visual mesh filename=package://vox_description/meshes/r1_link.stl
- link rf2_link: geometry collision mesh filename=package://vox_description/meshes/r2_link.stl; visual mesh filename=package://vox_description/meshes/r2_link.stl
- link rf3_link: geometry collision mesh filename=package://vox_description/meshes/r3_link.stl; visual mesh filename=package://vox_description/meshes/r3_link.stl
- link rf4_link: geometry collision mesh filename=package://vox_description/meshes/r4_link.stl; visual mesh filename=package://vox_description/meshes/r4_link.stl
- link rf5_link: geometry collision mesh filename=package://vox_description/meshes/r5_link.stl; visual mesh filename=package://vox_description/meshes/r5_link.stl
- link rf6_link: geometry collision mesh filename=package://vox_description/meshes/r6_link.stl; visual mesh filename=package://vox_description/meshes/r6_link.stl
- link rf7_link: geometry collision mesh filename=package://vox_description/meshes/r7_link.stl; visual mesh filename=package://vox_description/meshes/r7_link.stl
- link rf8_link: geometry collision mesh filename=package://vox_description/meshes/r8_link.stl; visual mesh filename=package://vox_description/meshes/r8_link.stl
- link rf9_link: geometry collision mesh filename=package://vox_description/meshes/r9_link.stl; visual mesh filename=package://vox_description/meshes/r9_link.stl
- link rl10_link: geometry collision mesh filename=package://vox_description/meshes/r10_link.stl; visual mesh filename=package://vox_description/meshes/r10_link.stl
- link rl1_link: geometry collision mesh filename=package://vox_description/meshes/r1_link.stl; visual mesh filename=package://vox_description/meshes/r1_link.stl
- link rl2_link: geometry collision mesh filename=package://vox_description/meshes/r2_link.stl; visual mesh filename=package://vox_description/meshes/r2_link.stl
- link rl3_link: geometry collision mesh filename=package://vox_description/meshes/r3_link.stl; visual mesh filename=package://vox_description/meshes/r3_link.stl
- link rl4_link: geometry collision mesh filename=package://vox_description/meshes/r4_link.stl; visual mesh filename=package://vox_description/meshes/r4_link.stl
- link rl5_link: geometry collision mesh filename=package://vox_description/meshes/r5_link.stl; visual mesh filename=package://vox_description/meshes/r5_link.stl
- link rl6_link: geometry collision mesh filename=package://vox_description/meshes/r6_link.stl; visual mesh filename=package://vox_description/meshes/r6_link.stl
- link rl7_link: geometry collision mesh filename=package://vox_description/meshes/r7_link.stl; visual mesh filename=package://vox_description/meshes/r7_link.stl
- link rl8_link: geometry collision mesh filename=package://vox_description/meshes/r8_link.stl; visual mesh filename=package://vox_description/meshes/r8_link.stl
- link rl9_link: geometry collision mesh filename=package://vox_description/meshes/r9_link.stl; visual mesh filename=package://vox_description/meshes/r9_link.stl
- link rr10_link: geometry collision mesh filename=package://vox_description/meshes/r10_link.stl; visual mesh filename=package://vox_description/meshes/r10_link.stl
- link rr1_link: geometry collision mesh filename=package://vox_description/meshes/r1_link.stl; visual mesh filename=package://vox_description/meshes/r1_link.stl
- link rr2_link: geometry collision mesh filename=package://vox_description/meshes/r2_link.stl; visual mesh filename=package://vox_description/meshes/r2_link.stl
- link rr3_link: geometry collision mesh filename=package://vox_description/meshes/r3_link.stl; visual mesh filename=package://vox_description/meshes/r3_link.stl
- link rr4_link: geometry collision mesh filename=package://vox_description/meshes/r4_link.stl; visual mesh filename=package://vox_description/meshes/r4_link.stl
- link rr5_link: geometry collision mesh filename=package://vox_description/meshes/r5_link.stl; visual mesh filename=package://vox_description/meshes/r5_link.stl
- link rr6_link: geometry collision mesh filename=package://vox_description/meshes/r6_link.stl; visual mesh filename=package://vox_description/meshes/r6_link.stl
- link rr7_link: geometry collision mesh filename=package://vox_description/meshes/r7_link.stl; visual mesh filename=package://vox_description/meshes/r7_link.stl
- link rr8_link: geometry collision mesh filename=package://vox_description/meshes/r8_link.stl; visual mesh filename=package://vox_description/meshes/r8_link.stl
- link rr9_link: geometry collision mesh filename=package://vox_description/meshes/r9_link.stl; visual mesh filename=package://vox_description/meshes/r9_link.stl
